Commit message: Enhance robot simulation setup by adding RViz configuration and lidar sensor definition, and updating launch files for improved simulation time handling.

File: my_robot_description/urdf/my_robot.urdf.xacro (robot description, xacro)
@@ -1,14 +1,8 @@
 <?xml version="1.0"?>
-<robot name="my_robot"  xmlns:xacro="http://ros.org/wiki/xacro">
+<robot name="my_robot" xmlns:xacro="http://www.ros.org/wiki/xacro">
   <xacro:include filename="common_properties.xacro"/>
   <xacro:include filename="mobile_base.xacro"/>
   <xacro:include filename="mobile_base_gazebo.xacro"/>
-  <xacro:include filename="arm.xacro"/>
-  <xacro:include filename="arm_gazebo.xacro"/>
   <xacro:include filename="camera.xacro"/>
-  <joint name="arm_to_baselink " type="fixed">
-    <parent link="base_link"/>
-    <child link="arm_base_link"/>
-    <origin xyz="${base_length/4} 0 ${base_height}" rpy="0 0 0"/>
-  </joint>
+  <xacro:include filename="lidar_sensor.xacro"/>
 </robot>
