Commit message: added nav2 , slam praram , maps

File: my_robot_description/urdf/lidar_sensor.xacro (robot description, xacro)
@@ -1,19 +1,17 @@
 <?xml version="1.0"?>
 <robot xmlns:xacro="http://www.ros.org/wiki/xacro">
-    <!-- Add your lidar sensor definition here -->
     <link name="lidar_link">
         <visual>
             <geometry>
-                <cylinder radius="0.05" length="0.1" />
+                <cylinder radius="0.035" length="0.040" />
             </geometry>
             <material name="red" />
         </visual>
-        <origin xyz="0 0 0" rpy="0 0 0"/>
         <collision>
             <geometry>
-                <cylinder radius="0.05" length="0.1" />
+                <cylinder radius="0.035" length="0.040" />
             </geometry>
         </collision>
-        <xacro:box_inertial m="0.1" l="0.1" w="0.1" h="0.1"
+        <xacro:box_inertial m="0.1" l="0.07" w="0.07" h="0.04"
                            xyz="0 0 0" rpy="0 0 0" />
     </link>
@@ -21,40 +19,39 @@
         <parent link="base_link" />
         <child link="lidar_link" />
-        <!-- Fixed the syntax error: added missing closing parenthesis -->
-        <origin xyz="${base_length/4.0} 0 ${base_height + 0.05}" rpy="0 0 0" />
+        <origin xyz="${base_length/4.0} 0 ${base_height + 0.02}" rpy="0 0 0" />
     </joint>
-    <!-- Gazebo plugin for RPLiDAR A1 -->
     <gazebo reference="lidar_link">
         <material>Gazebo/Red</material>
-        <sensor type="ray" name="rplidar_a1_sensor">
+        <sensor type="ray" name="rplidar_sensor">
             <pose>0 0 0 0 0 0</pose>
             <visualize>true</visualize>
-            <update_rate>10</update_rate>
+            <update_rate>5.5</update_rate>
             <ray>
                 <scan>
                     <horizontal>
-                        <!-- RPLiDAR A1 specifications -->
                         <samples>360</samples>
                         <resolution>1</resolution>
-                        <min_angle>-3.141592654</min_angle>
-                        <max_angle>3.141592654</max_angle>
+                        <min_angle>-3.14159</min_angle>
+                        <max_angle>3.14159</max_angle>
                     </horizontal>
                 </scan>
                 <range>
-                    <!-- RPLiDAR A1 range specifications -->
-                    <min>0.15</min>
-                    <max>12.0</max>
-                    <resolution>0.01</resolution>
+                    <min>0.12</min>
+                    <max>3.5</max>
+                    <resolution>0.015</resolution>
                 </range>
                 <noise>
-                    <!-- Realistic noise for RPLiDAR A1 -->
                     <type>gaussian</type>
                     <mean>0.0</mean>
-                    <stddev>0.02</stddev>
+                    <stddev>0.01</stddev>
                 </noise>
             </ray>
-            <plugin name="gazebo_ros_rplidar_a1_controller" filename="libgazebo_ros_laser.so">
-                <topicName>/scan</topicName>
-                <frameName>lidar_link</frameName>
+            <plugin name="gazebo_ros_ray_sensor" filename="libgazebo_ros_ray_sensor.so">
+                <ros>
+                    <namespace>/</namespace>
+                    <remapping>~/out:=/scan</remapping>
+                </ros>
+                <output_type>sensor_msgs/LaserScan</output_type>
+                <frame_name>lidar_link</frame_name>
             </plugin>
         </sensor>
